Commit message: changes controller from diff drive gazebo plugin to diff_drive_controller pkg

File: robodrive_description/urdf/robodrive/macro.controller.xacro (robot description, xacro)
@@ -1,5 +1,5 @@
 <?xml version="1.0"?>
 <robot xmlns:xacro="http://www.ros.org/wiki/xacro" name="robodrive">
-    <xacro:macro name="robodrive_diff_drive">
+<!--     <xacro:macro name="robodrive_diff_drive">
     <gazebo>
         <plugin name="differential_drive_controller" filename="libgazebo_ros_diff_drive.so">
@@ -25,4 +25,29 @@
         </plugin>
     </gazebo>
+    </xacro:macro> -->
+    <xacro:macro name="robodrive_diff_drive">
+    <gazebo>
+        <plugin name="diff_drive_controller" filename="libgazebo_ros_control.so"/>
+    </gazebo>
+    <transmission name="left_wheel_trans">
+        <type>transmission_interface/SimpleTransmission</type>
+        <joint name="joint_wheel_left">
+            <hardwareInterface>hardware_interface/VelocityJointInterface</hardwareInterface>
+        </joint>
+        <actuator name="left_wheel_motor">
+        <hardwareInterface>VelocityJointInterface</hardwareInterface>
+        <mechanicalReduction>1</mechanicalReduction>
+        </actuator>
+    </transmission>
+    <transmission name="right_wheel_trans">
+        <type>transmission_interface/SimpleTransmission</type>
+        <joint name="joint_wheel_right">
+        <hardwareInterface>hardware_interface/VelocityJointInterface</hardwareInterface>
+        </joint>
+        <actuator name="right_wheel_motor">
+        <hardwareInterface>VelocityJointInterface</hardwareInterface>
+        <mechanicalReduction>1</mechanicalReduction>
+        </actuator>
+    </transmission>7
     </xacro:macro>
 </robot>
